Commit message: feat: Add rgbd camera

File: slam_project/urdf/xbot.xacro (robot description, xacro)
@@ -8,10 +8,16 @@
     <child link="chassis" />
   </joint>
-  <joint type="fixed" name="camera_joint">
+<joint name="camera_joint" type="fixed">
+   <origin xyz="0 0 0" rpy="-1.5707 0 -1.5707"/>
+   <parent link="camera_link"/>
+   <child link="rgbd_frame"/>
+</joint>
+<link name="rgbd_frame"/>
+  <joint type="fixed" name="camera_base_joint">
     <origin xyz="0.175 0 0" rpy="0 0 0"/>
-    <child link="camera"/>
+    <child link="camera_link"/>
     <parent link="sensor_base"/>
   </joint>
- <link name='camera'>
+ <link name='camera_link'>
     <inertial>
       <mass value="0.1"/>

Commit message: fix: Correct topic names and link names.
Mapping ready with laser scan.

File: slam_project/urdf/xbot.xacro (robot description, xacro)
@@ -11,7 +11,7 @@
    <origin xyz="0 0 0" rpy="-1.5707 0 -1.5707"/>
    <parent link="camera_link"/>
-   <child link="rgbd_frame"/>
+   <child link="camera_rgbd_frame"/>
 </joint>
-<link name="rgbd_frame"/>
+<link name="camera_rgbd_frame"/>
   <joint type="fixed" name="camera_base_joint">
     <origin xyz="0.175 0 0" rpy="0 0 0"/>
